Commit message: Updated hardware interface, still need to setup hid comms

File: src/xarm_description/urdf/XArm.xacro (robot description, xacro)
@@ -4,5 +4,5 @@
 <xacro:include filename="$(find xarm_description)/urdf/materials.xacro" />
 <xacro:include filename="$(find xarm_description)/urdf/XArm.trans" />
-<xacro:include filename="$(find xarm_description)/urdf/XArm.gazebo" />
+<!-- <xacro:include filename="$(find xarm_description)/urdf/XArm.gazebo" /> -->
 <xacro:include filename="$(find xarm_description)/urdf/ros2_control.xacro" />
  <link name="xarm_base_link">
@@ -165,3 +165,4 @@
         <child link="xarm_2_link" />
     </joint>
+<xacro:XArm name="XArmHardware" prefix=""/>
 </robot>

File: src/xarm_description/urdf/ros2_control.xacro (robot description, xacro)
@@ -1,10 +1,13 @@
 <?xml version="1.0"?>
 <robot xmlns:xacro="http://www.ros.org/wiki/xacro">
-    <xacro:macro name="XArm_ros2_control" params="name initial_positions_file">
+    <xacro:macro name="XArm" params="name prefix">
         <!-- <xacro:property name="initial_positions" value="${load_yaml(initial_positions_file)['initial_positions']}"/> -->
-        <ros2_control name="XArmSystemHardware" type="system">
+        <ros2_control name="${name}" type="system">
         <hardware>
             <!-- By default, set up controllers for simulation. This won't work on real hardware -->
-            <plugin>xarm_description/XArmSystemHardware</plugin>
+            <plugin>xarm_hardware/XArmSystemHardware</plugin>
+            <parameters>$(find xarm_description)/config/my_controllers.yaml</parameters>
+            <param name="example_param_hw_start_duration_sec">2.0</param>
+            <param name="example_param_hw_stop_duration_sec">3.0</param>
         </hardware>
             <joint name="xarm_6_joint">

File: src/xarm_moveit_config/config/XArm.urdf.xacro (robot description, xacro)
@@ -5,5 +5,5 @@
     <xacro:include filename="$(find xarm_description)/urdf/XArm.xacro" />
     <!-- Import control_xacro -->
-    <xacro:include filename="XArm.ros2_control.xacro" />
+    <!-- <xacro:include filename="XArm.ros2_control.xacro" /> -->
     <!-- <xacro:XArm_ros2_control name="FakeSystem" initial_positions_file="$(arg initial_positions_file)"/> -->
 </robot>
